Commit message: Update robot model file

File: lerobot_ws/install/lerobot_description/share/lerobot_description/urdf/robot.urdf (robot description, URDF)
Before this commit: robot lerobot, 5 links, 4 joints
Links:
- removed link dummy_link
- removed link link1
- removed link link2
- removed link tool
- added link forearm_link; collision box size=0.020 0.014 0.090; collision box size=0.032 0.032 0.032
- added link gripper_base_link; collision box size=0.015 0.080 0.015; collision box size=0.040 0.038 0.040
- added link gripper_left_finger_link; collision box size=0.045 0.010 0.014; collision box size=0.070 0.010 0.014
- added link gripper_right_finger_link; collision box size=0.045 0.010 0.014; collision box size=0.070 0.010 0.014
- added link shoulder_link; collision box size=0.04 0.038 0.055; visual box size=0.04 0.038 0.055
- added link tcp_link
- added link upper_arm_link; collision box size=0.022 0.014 0.130; collision box size=0.038 0.038 0.040
- link base_link: geometry collision cylinder length=0.008 radius=0.075; collision cylinder length=0.012 radius=0.065
Joints:
- added joint gripper_left_finger_joint: type revolute, parent gripper_base_link, child gripper_left_finger_link, origin xyz=0.055 -0.035 0 rpy=0 0 0, axis 0 0 1, limit lower=-0.6 upper=0.0 effort=10 velocity=1.0
- added joint gripper_right_finger_joint: type revolute, parent gripper_base_link, child gripper_right_finger_link, origin xyz=0.055 0.035 0 rpy=0 0 0, axis 0 0 1, limit lower=0.0 upper=0.6 effort=10 velocity=1.0, mimic joint=gripper_left_finger_joint multiplier=-1.0 offset=0.0
- added joint gripper_tcp_joint: type fixed, parent gripper_base_link, child tcp_link, origin xyz=0.110 0 0
- joint joint1: child dummy_link -> shoulder_link; limit lower=-3.1416 upper=3.1416 effort=10 velocity=1.0 -> lower=-3.1416 upper=3.1416 effort=15 velocity=1.0; origin xyz=0 0 0.025 -> xyz=0 0 0.006
- joint joint2: child link1 -> upper_arm_link; limit lower=-1.5708 upper=1.5708 effort=10 velocity=1.0 -> lower=-1.5708 upper=1.5708 effort=15 velocity=1.0; origin xyz=0 0 0 -> xyz=0 0 0.054; parent dummy_link -> shoulder_link
- joint joint3: child link2 -> forearm_link; origin xyz=0 0 0.1 -> xyz=0 0 0.165; parent link1 -> upper_arm_link
- joint joint4: axis 0 1 0 -> (none); child tool -> gripper_base_link; limit lower=-0.7854 upper=0.7854 effort=10 velocity=1.0 -> (none); origin xyz=0 0 0.1 -> xyz=0 0 0.112 rpy=0 -1.5708 0; parent link2 -> forearm_link; type revolute -> fixed
